File: Shields/Empty_Template/Eagle/Shield_Empty.brd (EAGLE design)
At the start: 31.9 x 17.8 mm, 3 parts

Commit message: Updated readme and removed TinyPICO logo from shield template
Parts:
- moved LOGO1 6.69 mm to (27.6, 8.88)
